Commit message: updated height about ground dimensions

File: urdf/warehouse_bot.urdf (robot description, URDF)
Before this commit: robot warehouse_bot, 2 links, 1 joints
Joints:
- joint base_footprint_to_base_link: origin xyz=0.0 0.0 1.0 -> xyz=0.0 0.0 0.05

Commit message: Added in left and right wheels

File: urdf/warehouse_bot.urdf (robot description, URDF)
Before this commit: robot warehouse_bot, 2 links, 1 joints
Links:
- added link wheel_left_link; visual mesh filename=package://warehousebot_description/meshes/left_wheel.stl scale=0.01 0.01 0.01
- added link wheel_right_link; visual mesh filename=package://warehousebot_description/meshes/right_wheel.stl scale=0.01 0.01 0.01
Joints:
- added joint wheel_left_joint: type fixed, parent base_link, child wheel_left_link, origin xyz=0 0.159974 0.0485 rpy=1.57 0 0, axis 0 0 1
- added joint wheel_right_joint: type fixed, parent base_link, child wheel_right_link, origin xyz=0 -0.159974 0.0485 rpy=1.57 0 0, axis 0 0 1

Commit message: Added in laser frame

File: urdf/warehouse_bot.urdf (robot description, URDF)
Before this commit: robot warehouse_bot, 4 links, 3 joints
Links:
- added link laser_front; visual mesh filename=package://warehousebot_description/meshes/sick_tim_571.stl
Joints:
- added joint base_link_to_laser_front: type fixed, parent base_link, child laser_front, origin xyz=0.169 0.0 0.035856 rpy=3.142 0.0 0.0

Commit message: Renamed base_scan to base_laser

File: urdf/warehouse_bot.urdf (robot description, URDF)
Before this commit: robot warehouse_bot, 5 links, 4 joints
Links:
- removed link laser_front
- added link base_laser; visual mesh filename=package://warehousebot_description/meshes/sick_tim_571.stl
Joints:
- joint base_link_to_laser_front: child laser_front -> base_laser
