Commit message: updated launch file and warehousebot urdf

File: urdf/warehouse_bot.urdf.xacro (robot description, xacro)
@@ -2,4 +2,6 @@
 <robot name="warehouse_bot"
   xmlns:xacro="http://ros.org/wiki/xacro">
+  <xacro:include filename="$(find warehousebot_description)/urdf/_d435.urdf.xacro" />
+  <xacro:arg name="use_nominal_extrinsics" default="true"/>
   <link name="base_laser">
     <visual>
@@ -39,4 +41,7 @@
     </visual>
   </link>
+  <xacro:sensor_d435 parent="base_link" use_nominal_extrinsics="$(arg use_nominal_extrinsics)">
+    <origin xyz="0.19065 0 0.254" rpy="0 0 0"/>
+  </xacro:sensor_d435>
   <joint name="base_footprint_to_base_link" type="fixed">
     <parent link="base_footprint"/>
