Commit message: Added in frame for imu

File: urdf/_d435.urdf.xacro (robot description, xacro)
@@ -69,4 +69,11 @@
       </inertial>
     </link>
+    <!-- frames for imu -->
+    <link name="${name}_imu_optical_frame" />
+    <joint name="${name}_imu_joint" type="fixed">
+      <origin xyz = "-0.01174 -0.00552 0.0051" rpy = "0 0 0" />
+      <parent link="${name}_link" />
+      <child link="${name}_imu_optical_frame" />
+    </joint>
     <!-- Use the nominal extrinsics between camera frames if the calibrated extrinsics aren't being published. e.g. running the device in simulation  -->
     <xacro:if value="${use_nominal_extrinsics}">

Commit message: updated rotation of imu frame

File: urdf/_d435.urdf.xacro (robot description, xacro)
@@ -72,5 +72,5 @@
     <link name="${name}_imu_optical_frame" />
     <joint name="${name}_imu_joint" type="fixed">
-      <origin xyz = "-0.01174 -0.00552 0.0051" rpy = "0 0 0" />
+      <origin xyz = "-0.01174 -0.00552 0.0051" rpy = "-1.571 0 -1.571" />
       <parent link="${name}_link" />
       <child link="${name}_imu_optical_frame" />
